File: lab6/completefilter.brd (EAGLE design)
At the start: 80 x 34 mm, 23 parts, among them IC1 LM386N-1, IC2 LM386N-1, IC3 LM386N-1

Commit message: Merge issue in lab6.tex resolved and compiled.
Parts:
- moved R2 3.81 mm to (47.0, 26.7)
- moved C2 2.54 mm to (64.8, 15.2)
- moved C5 2.54 mm to (52.1, 15.2)
- moved C6 2.54 mm to (34.3, 15.2)
- moved C7 2.54 mm to (39.4, 15.2)
- moved R3 2.54 mm to (47.0, 15.2)
- moved C1 2.54 mm to (59.7, 21.6)
- moved C3 2.54 mm to (47.0, 21.6)
- moved C4 2.54 mm to (52.1, 21.6)
- moved R1 2.54 mm to (64.8, 21.6)
- moved R4 2.54 mm to (39.4, 21.6)
- moved SJ1 1.27 mm to (16.5, 15.2), flipped to the bottom, turned to 180 degrees
Routing:
- net GND: track 55.3 -> 50.1 mm
- net SIGIN: track 53.6 -> 50.1 mm
- net LP: track 6.22 -> 3.68 mm
- net HP: track 6.22 -> 3.68 mm
- net BP: track 6.22 -> 3.68 mm
- net N$2: track 8.61 -> 7.34 mm
- net N$7: track 18.4 -> 17.9 mm
Other:
- board size 80 x 34 mm -> 80 x 30.1 mm
